File: FInalCircuits/AUV/SideMotors/SideMotors.kicad_sch (KiCad schematic)
At the start: 5 parts, among them J2 Motor Controller, J3 TWI, U1 ATtiny1627-M

Commit message: First draft of Design portion of the FinalReport
Parts:
- U1: value ATtiny1627-M -> Side Motors
Changed lines of the file:
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@@
 			)
 		)
-		(property "Value" "ATtiny1627-M"
+		(property "Value" "Side Motors"
 			(at 72.0441 45.72 0)
 			(effects
